Commit message: [urdf] Add visuals of vacuum pad and camera d435i.

File: urdf/ur5e.urdf (robot description, URDF)
Before this commit: robot ur5e_robot, 11 links, 10 joints
Links:
- added link d435i; visual mesh filename=package://mc_ur5e_description/urdf/meshes/d435i_0.stl; visual mesh filename=package://mc_ur5e_description/urdf/meshes/d435i_1.stl
- added link vacuum_pad; visual mesh filename=package://mc_ur5e_description/urdf/meshes/SMC-ZP3P-50PTSF.s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 scale=0.001 0.001 0.001
Joints:
- added joint tool0-d435i: type fixed, parent tool0, child d435i, origin xyz=0 0.05 0 rpy=0 0 0
- added joint tool0-vacuum_pad: type fixed, parent tool0, child vacuum_pad

Commit message: [urdf] Limit joint range.
This joint range limit is suitable for handling a region with negative X-coordinates in the world frame.

File: urdf/ur5e.urdf (robot description, URDF)
Before this commit: robot ur5e_robot, 13 links, 12 joints
Joints:
- joint elbow_joint: limit lower=-3.141592653589793 upper=3.141592653589793 effort=150.0 velocity=3.141592653589793 -> lower=-3.141592653589793 upper=0.0 effort=150.0 velocity=3.141592653589793
- joint shoulder_pan_joint: limit lower=-6.283185307179586 upper=6.283185307179586 effort=150.0 velocity=3.141592653589793 -> lower=-1.5707963267948966 upper=1.5707963267948966 effort=150.0 velocity=3.141592653589793
